File: hardware/kicad/Bachelorprojekt.kicad_sch (KiCad schematic)
At the start: 37 parts, among them J1 Screw_Terminal_01x02, J10 Conn_01x02_Pin, J11 Conn_01x02_Pin, J12 Conn_01x02_Pin, J13 Conn_01x02_Pin, J14 Conn_01x02_Pin, J15 Conn_01x02_Pin, J16 Conn_01x02_Pin, J2 Screw_Terminal_01x03, J3 Conn_01x04_Pin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

Commit message: Opdater kalibrering og pulsoximeterdata
Other:
- note added: "10k ohm"
- note added: "1M ohm"
- note added: "2.1 Mohm"
- note added: "39k ohm"
- note added: "G = 1 + 39k/10k = 4.9"
- note added: "fc = 1/(2*3.14*1e6*1e-9) ~= 159 Hz"
- note removed: "100k ohm"
- note removed: "1k ohm"
- note removed: "20k ohm"
- note removed: "56k ohm"
Changed lines of the file:
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@@
 		)
 	)
-	(text "1k ohm"
+	(text "10k ohm"
 		(exclude_from_sim no)
 		(at 209.804 155.702 0)
@@
 		)
 	)
-	(text "20k ohm"
+	(text "39k ohm"
 		(exclude_from_sim no)
 		(at 235.712 154.94 0)
@@
 		)
 	)
-	(text "56k ohm"
+	(text "1M ohm"
 		(exclude_from_sim no)
 		(at 208.026 53.594 0)
@@
 		(exclude_from_sim no)
 		(at 37.338 74.168 0)
+		(effects
+			(font
+				(size 1.27 1.27)
+			)
+		)
+	)
+	(text "fc = 1/(2*3.14*1e6*1e-9) ~= 159 Hz"
+		(exclude_from_sim no)
+		(at 203.454 68.834 0)
 		(effects
 			(font
@@
 		)
 	)
+	(text "G = 1 + 39k/10k = 4.9"
+		(exclude_from_sim no)
+		(at 264.668 142.494 0)
+		(effects
+			(font
+				(size 1.27 1.27)
+			)
+		)
+	)
 	(text "330k ohm"
 		(exclude_from_sim no)
@@
 		)
 	)
-	(text "100k ohm\n"
+	(text "2.1 Mohm\n"
 		(exclude_from_sim no)
 		(at 106.934 25.654 0)
@@
 		)
 	)
-	(text "56k ohm"
+	(text "1M ohm"
 		(exclude_from_sim no)
 		(at 225.044 53.594 0)

Commit message: Tilføj endelige kalibreringsmålinger og hardwarefiler
Other:
- note added: "2.21 Mohm"
- note removed: "2.1 Mohm"
- note removed: "fc = 1/(2*3.14*1e6*1e-9) ~= 159 Hz"
Changed lines of the file:
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@@
-		)
-	)
-	(text "fc = 1/(2*3.14*1e6*1e-9) ~= 159 Hz"
-		(exclude_from_sim no)
-		(at 203.454 68.834 0)
-		(effects
-			(font
-				(size 1.27 1.27)
-			)
 		)
 	)
@@
 		)
 	)
-	(text "2.1 Mohm\n"
+	(text "2.21 Mohm\n"
 		(exclude_from_sim no)
 		(at 106.934 25.654 0)
